Commit message: reduced gazebo friction

File: workstation/pupper_description/motor.xacro (robot description, xacro)
@@ -40,5 +40,5 @@
             <xacro:insert_block name = "revolute_origin"/>
             <limit upper = "1e10" lower = "-1e10" effort = "1e6" velocity = "1e6"/>
-            <dynamics damping = "0.2" friction = "0.3"/>
+            <dynamics damping = "0.01" friction = "0.0001"/>
             <axis xyz = "${axis}"/>
         </joint>
