Commit message: kd and kp added to feet collisions

File: workstation/pupper_description/left_leg.xacro (robot description, xacro)
@@ -113,4 +113,16 @@
         </link>
         <xacro:if value = "${full_urdf}">
+        <gazebo reference="${name}_left_foot">
+            <collision>
+                <surface>
+                    <contact>
+                        <ode>
+                            <kp>1e15</kp>
+                            <kd>1e13</kd>
+                        </ode>
+                    </contact>
+                </surface>
+            </collision>
+        </gazebo>
         <gazebo reference="${lowerName}">
             <collision>

File: workstation/pupper_description/right_leg.xacro (robot description, xacro)
@@ -113,4 +113,16 @@
         </link>
         <xacro:if value = "${full_urdf}">
+        <gazebo reference="${name}_right_foot">
+            <collision>
+                <surface>
+                    <contact>
+                        <ode>
+                            <kp>1e15</kp>
+                            <kd>1e13</kd>
+                        </ode>
+                    </contact>
+                </surface>
+            </collision>
+        </gazebo>
         <gazebo reference="${lowerName}">
             <collision>

Commit message: dynamic model and urdf redone using solidworks

File: workstation/pupper_description/left_leg.xacro (robot description, xacro)
@@ -27,9 +27,9 @@
                 </geometry>
             </visual>
-            <collision name = "${hubName}_collision">
+            <!-- <collision name = "${hubName}_collision">
                 <geometry>
                     <mesh filename = "${CollisionPath}/Leg/assembly_hip_left_simplified.dae" scale = "${meshScale_meters}"/>
                 </geometry>
-            </collision>
+            </collision> -->
             </xacro:if>
         </link>
@@ -57,7 +57,11 @@
             </visual>
             <collision name = "${upperName}_collision">
+                <origin xyz = "0.0 0.0233 -0.080" rpy = "${PI/2} 0 0"/>
                 <geometry>
+                    <cylinder radius = "0.0095" length = "0.045"/>
+                </geometry>
+                <!-- <geometry>
                     <mesh filename = "${CollisionPath}/Leg/assembly_upper_link_left_simplified.dae" scale = "${meshScale_meters}"/>
-                </geometry>
+                </geometry> -->
             </collision>
             </xacro:if>
@@ -86,7 +90,11 @@
             </visual>
             <collision name = "${lowerName}_collision">
+                <origin xyz = "0.0 -0.0095 -.11" />
                 <geometry>
-                    <mesh filename = "${CollisionPath}/Leg/assembly_lower_link_left_simplified.dae" scale = "${meshScale_meters}"/>
+                    <box size = "0.00001 0.00001 0.00001"/>
                 </geometry>
+                <!-- <geometry> -->
+                <!--     <mesh filename = "${CollisionPath}/Leg/assembly_lower_link_left_simplified.dae" scale = "${meshScale_meters}"/> -->
+                <!--  </geometry> -->
             </collision>
             </xacro:if>
@@ -98,7 +106,6 @@
                     <contact>
                         <ode>
-                            <xacro:insert_block name = "contact_kp" /> <!-- <kp>1e15</kp> -->
-                            <xacro:insert_block name = "contact_kd" /> <!-- <kd>1e13</kd> -->
-                            <!-- <min_depth>0.01</min_depth> -->
+                            <xacro:insert_block name = "contact_kp" />
+                            <xacro:insert_block name = "contact_kd" />
                         </ode>
                     </contact>

File: workstation/pupper_description/pupper.urdf (robot description, URDF)
Before this commit: robot pupper, 13 links, 12 joints
Links:
- link back_left_lower_link: geometry collision sphere ; visual mesh filename=package://workstation/pupper_description/Pupper_STL/Leg/ass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 scale=1.0 1.0 1.0
- link front_left_lower_link: geometry collision sphere ; visual mesh filename=package://workstation/pupper_description/Pupper_STL/Leg/ass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 scale=1.0 1.0 1.0

File: workstation/pupper_description/pupper.urdf.xacro (robot description, xacro)
@@ -131,11 +131,11 @@
     <!-- +++++++++++++++++++ -->
     <xacro:property name = "contact_kp">
-        <kp>1e15</kp>
+        <kp>1e6</kp>
     </xacro:property>
     <xacro:property name = "contact_kd">
-        <kp>1.5e14</kp>
+        <kd>1</kd>
     </xacro:property>
     <xacro:property name = "joint_friction">
-        <dynamics damping = "0.01" friction = "0.0001"/>
+        <dynamics damping = "0.001" friction = "0.17"/>
     </xacro:property>
     <!-- Connect the plugin -->
@@ -167,7 +167,11 @@
         </visual>
         <collision name = "bottom_PCB_collision">
+            <origin xyz = "0.0 0.0 0.04355" rpy = "0 0 0"/>
             <geometry>
+                <box size = "0.264 0.124 0.0901"/>
+            </geometry>
+            <!-- <geometry>
                 <mesh filename = "${CollisionPath}/Body/assembly_body_simplified.dae" scale = "${meshScale_meters}"/>
-            </geometry>
+            </geometry> -->
         </collision>
         </xacro:if>

File: workstation/pupper_description/right_leg.xacro (robot description, xacro)
@@ -27,9 +27,9 @@
                 </geometry>
             </visual>
-            <collision name = "${hubName}_collision">
+            <!-- <collision name = "${hubName}_collision">
                 <geometry>
                     <mesh filename = "${CollisionPath}/Leg/assembly_hip_right_simplified.dae" scale = "${meshScale_meters}"/>
                 </geometry>
-            </collision>
+            </collision> -->
             </xacro:if>
         </link>
@@ -57,7 +57,11 @@
             </visual>
             <collision name = "${upperName}_collision">
+                <origin xyz = "0.0 -0.0233 -0.080" rpy = "${PI/2} 0 0"/>
                 <geometry>
+                    <cylinder radius = "0.0095" length = "0.045"/>
+                </geometry>
+                <!-- <geometry>
                     <mesh filename = "${CollisionPath}/Leg/assembly_upper_link_right_simplified.dae" scale = "${meshScale_meters}"/>
-                </geometry>
+                </geometry> -->
             </collision>
             </xacro:if>
@@ -86,6 +90,7 @@
             </visual>
             <collision name = "${lowerName}_collision">
+                <origin xyz = "0.0 0.0095 -.11" />
                 <geometry>
-                    <mesh filename = "${CollisionPath}/Leg/assembly_lower_link_right_simplified.dae" scale = "${meshScale_meters}"/>
+                    <box size = "0.00001 0.00001 0.00001"/>
                 </geometry>
             </collision>
@@ -98,7 +103,6 @@
                     <contact>
                         <ode>
-                            <xacro:insert_block name = "contact_kp" /> <!-- <kp>1e15</kp> -->
-                            <xacro:insert_block name = "contact_kd" /> <!-- <kd>1e13</kd> -->
-                            <!-- <min_depth>0.01</min_depth> -->
+                            <xacro:insert_block name = "contact_kp" />
+                            <xacro:insert_block name = "contact_kd" />
                         </ode>
                     </contact>
